File: bno055/bno055.kicad_pcb (KiCad board)
At the start: 4 copper layers, 11 parts, among them U1 BNO055, Y1 NX3215SA-32.768K-STD-MUA-14

Commit message: [Rushil] added block of ds3231_rtc
Parts:
- added R2: 10k, Resistor_SMD:R_0603_1608Metric, F.Cu at (113.8, 78.7)
- added R5: 10k, Resistor_SMD:R_0603_1608Metric, F.Cu at (116.9, 78.7)
Routing:
- net /block_bno055/+3V3: track 6.62 -> 21.3 mm, vias 0 -> 2
- net /block_bno055/SDA: track 0.00 -> 5.61 mm
- net /block_bno055/SCL: track 0.00 -> 2.00 mm

Commit message: [Rushil] corrected pcb added information on both schematic and pcb user drawing correct circuit of bno055
Parts:
- removed TP1: TestPoint, Library:TestPoint_Pad_D1.5mm
- added D1: 1N4148WS, 1N4148WS:SOD323, F.Cu at (106.5, 75.0)
- added JP1: Jumper_2_Open, Jumper:SolderJumper-2_P1.3mm_Open_RoundedPad1.0x1.5mm, F.Cu at (106.5, 78.4)
- added R6: 10k, Resistor_SMD:R_0603_1608Metric, F.Cu at (106.5, 76.4)
- moved C3 0.79 mm to (106.5, 73.5)
- moved R3 0.79 mm to (106.5, 72.0)
Connections:
- U1 pad 10: Net-(U1-BL_IND) -> unconnected-(U1-BL_IND-Pad10)
- U1 pad 11: /block_bno055/NRESET -> Net-(U1-~{RESET})
Routing:
- net /block_bno055/+3V3: track 21.3 -> 14.0 mm, vias 2 -> 3
- net Net-(U1-~{RESET}): track 0.00 -> 3.47 mm
- net Net-(U1-BL_IND): track 3.31 -> 0.00 mm
- net Net-(JP1-B): track 1.97 -> 4.84 mm
- net /block_bno055/GND: track 6.96 -> 9.63 mm, vias 14 -> 19
- net Net-(U1-CAP): track 1.64 -> 2.43 mm
- net Net-(U1-PS0): track 1.62 -> 2.41 mm
- added copper zone on In2.Cu, net /block_bno055/+3V3
Other:
- board text added: "32.768 kHz RTC Crystal - Keep traces short and symmetric - No GND plane under crystal - C4, C5 = 22 pF load capacitors"
- board text added: "9-DOF absolute orientation sensor with onboard fusion"
- board text added: "BNO055 sensor Rule out area Layer 2 and 3"
- board text added: "Crystal Rule out area Layer 2 and 3"
- board text added: "Rule area under sensor and crystal avoid high current near the sensor and crystal"
- board text removed: "Rule area under sensor and crystal avoid high current near the sensor and crystal it is recommended to have no fill area under crystal of low frequency of such as . made a gnd ring around crystal"

Commit message: fixed BNO055
Connections:
- net /block_bno055/+3V3 renamed /block_bno055/3V3
Changed lines of the file:
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@@
 			(psa4output no)
 			(plot_black_and_white yes)
+			(plotinvisibletext no)
 			(sketchpadsonfab no)
 			(plotpadnumbers no)
@@
 	)
 	(net 0 "")
-	(net 1 "/block_bno055/+3V3")
+	(net 1 "/block_bno055/3V3")
 	(net 2 "/block_bno055/GND")
 	(net 3 "Net-(U1-CAP)")
@@
 			(layers "F.Cu" "F.Mask" "F.Paste")
 			(roundrect_rratio 0.25)
-			(net 1 "/block_bno055/+3V3")
+			(net 1 "/block_bno055/3V3")
 			(pintype "passive")
 		)
@@
 			(layers "F.Cu" "F.Mask" "F.Paste")
 			(roundrect_rratio 0.25)
-			(net 1 "/block_bno055/+3V3")
+			(net 1 "/block_bno055/3V3")
 			(pintype "passive")
 		)
@@
 			(size 0.254 0.675)
 			(layers "F.Cu" "F.Mask" "F.Paste")
-			(net 1 "/block_bno055/+3V3")
+			(net 1 "/block_bno055/3V3")
 			(pinfunction "VDD")
 			(pintype "power_in")
@@
 			(size 0.254 0.675)
 			(layers "F.Cu" "F.Mask" "F.Paste")
-			(net 1 "/block_bno055/+3V3")
+			(net 1 "/block_bno055/3V3")
 			(pinfunction "~{BOOT_LOAD_PIN}")
 			(pintype "input")
@@
 			(size 0.254 0.675)
 			(layers "F.Cu" "F.Mask" "F.Paste")
-			(net 1 "/block_bno055/+3V3")
+			(net 1 "/block_bno055/3V3")
 			(pinfunction "VDDIO")
 			(pintype "power_in")
@@
 			(layers "F.Cu" "F.Mask" "F.Paste")
 			(roundrect_rratio 0.25)
-			(net 1 "/block_bno055/+3V3")
+			(net 1 "/block_bno055/3V3")
 			(pintype "passive")
 		)
@@
 			(layers "F.Cu" "F.Mask" "F.Paste")
 			(roundrect_rratio 0.25)
-			(net 1 "/block_bno055/+3V3")
+			(net 1 "/block_bno055/3V3")
 			(pintype "passive")
 		)
@@
 			(layers "F.Cu" "F.Mask" "F.Paste")
 			(roundrect_rratio 0.25)
-			(net 1 "/block_bno055/+3V3")
+			(net 1 "/block_bno055/3V3")
 			(pintype "passive")
 		)
@@
 			(size 1 0.5)
 			(layers "F.Cu" "F.Mask")
-			(net 1 "/block_bno055/+3V3")
+			(net 1 "/block_bno055/3V3")
 			(pinfunction "A")
 			(pintype "passive")
@@
 		(tags "resistor")
 		(property "Reference" "R4"
-			(at -0.09 -1.23 90)
+			(at -0.35 -1.33 90)
 			(layer "F.SilkS")
 			(effects
@@
 	)
 	(gr_text "BNO055"
-		(at 104.5 69.5 0)
+		(at 103.9 69.8 0)
 		(layer "F.SilkS")
 		(effects
 			(font
-				(size 0.7 0.7)
+				(size 0.8 0.8)
 				(thickness 0.15)
 			)
@@
 	(zone
 		(net 1)
-		(net_name "/block_bno055/+3V3")
+		(net_name "/block_bno055/3V3")
 		(layer "In2.Cu")
 		(hatch edge 0.5)
