File: tmc2209/tmc2209.kicad_pcb (KiCad board)
At the start: 4 copper layers, 25 parts, among them J1 MOTOR CONNECTOR, U1 TMC2209-LA

Commit message: [Rushil] added some more info on silkscreen
Parts:
- moved R6 0.06 mm to (122.5, 68.4)
Other:
- board text added: "dir leds"
- board text added: "step led"
Changed lines of the file:
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@@
 		(tags "LED handsolder")
 		(property "Reference" "D1"
-			(at -2.575 0 180)
+			(at 2.725 0 180)
 			(layer "F.SilkS")
 			(effects
@@
 		(tags "capacitor")
 		(property "Reference" "C5"
-			(at 2.3 0 90)
+			(at 2 0 180)
 			(layer "F.SilkS")
 			(effects
@@
 	(footprint "Library:R_0805_2012Metric_Pad1.20x1.40mm_HandSolder"
 		(layer "F.Cu")
-		(at 122.53 68.5 90)
+		(at 122.53 68.44 90)
 		(descr "Resistor SMD 0805 (2012 Metric), square (rectangular) end terminal, IPC-7351 nominal with elongated pad for handsoldering. (Body size source: IPC-SM-782 page 72, https://www.pcb-3d.com/wordpress/wp-content/uploads/ipc-sm-782a_amendment_1_and_2.pdf), generated with kicad-footprint-generator")
 		(tags "resistor handsolder")
@@
 		)
 	)
+	(gr_text "step \nled\n"
+		(at 128.8 83 0)
+		(layer "F.SilkS")
+		(effects
+			(font
+				(size 0.7 0.7)
+				(thickness 0.153)
+				(bold yes)
+			)
+			(justify left bottom)
+		)
+	)
 	(gr_text "TMC2209"
-		(at 131 82 0)
+		(at 132.2 80.2 0)
+		(layer "F.SilkS")
+		(effects
+			(font
+				(size 0.7 0.7)
+				(thickness 0.153)
+				(bold yes)
+			)
+			(justify left bottom)
+		)
+	)
+	(gr_text "dir \nleds\n"
+		(at 128.8 73.8 0)
 		(layer "F.SilkS")
 		(effects
@@
 			(pts
 				(xy 125.74 71.26) (xy 126.2 70.8) (xy 130.79 70.8) (xy 131.02 71.03) (xy 131.02 72.12) (xy 130.86 72.28)
-				(xy 125.74 72.28) (xy 125.74 72.28)
+				(xy 125.74 72.28)
 			)
 		)
