File: esp32-s3-wroom-2/esp32-s3-wroom-2.kicad_sch (KiCad schematic)
At the start: 0 parts

Commit message: [Rushil] fixed block name of esp32 wroom
Other:
- sheet block_esp32-s3-wroom-2 renamed esp32-s3-wroom-2
Changed lines of the file:
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@@
 			(color 0 0 0 0.0000)
 		)
-		(property "Sheetname" "block_esp32-s3-wroom-2"
+		(property "Sheetname" "esp32-s3-wroom-2"
 			(at 83.82 52.6284 0)
 			(effects

Commit message: [Rushil] fixed block esp32 wroom
Other:
- sheet esp32-s3-wroom-2 ports: added 3V3; removed +3V3
Changed lines of the file:
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@@
 			)
 		)
-		(pin "+3V3" input
+		(pin "3V3" input
 			(at 83.82 58.42 180)
 			(effects
