File: lm2662m/block_lm2662m.kicad_sch (KiCad schematic)
At the start: 7 parts, among them J1 Jumper, U1 LM2662M

Commit message: [Rushil] changed vccn to vee
Connections:
- net VCCN renamed VEE
Other:
- note added: "LM2662M - Inverting Charge Pump Converter Function: - Generates a negative voltage (VEE(-VCC)) from a positive input supply (VCC) Operating Range: - Input Voltage (VCC): 1.5V to 5.5V - Output Current: Up to 200 mA (typical)"
- note removed: "LM2662M - Inverting Charge Pump Converter Function: - Generates a negative voltage (-VCC) from a positive input supply (VCC) Operating Range: - Input Voltage (VCC): 1.5V to 5.5V - Output Current: Up to 200 mA (typical)"
Changed lines of the file:
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@@
 		)
 	)
-	(text "LM2662M - Inverting Charge Pump Converter\nFunction:\n- Generates a negative voltage (-VCC) from a positive input supply (VCC)\nOperating Range:\n- Input Voltage (VCC): 1.5V to 5.5V\n- Output Current: Up to 200 mA (typical)\n\n"
+	(text "LM2662M - Inverting Charge Pump Converter\nFunction:\n- Generates a negative voltage (VEE(-VCC)) from a positive input supply (VCC)\nOperating Range:\n- Input Voltage (VCC): 1.5V to 5.5V\n- Output Current: Up to 200 mA (typical)\n\n"
 		(exclude_from_sim no)
 		(at 88.9 112.268 0)
@@
 		)
 	)
-	(hierarchical_label "VCCN"
+	(hierarchical_label "VEE"
 		(shape input)
 		(at 187.96 72.39 0)
