File: lm2662m/lm2662m.kicad_pcb (KiCad board)
At the start: 4 copper layers, 7 parts, among them J1 Jumper, U1 LM2662M

Commit message: [Rushil] changed vccn to vee
Connections:
- net /LM2662M/VCCN renamed /LM2662M/VEE
Other:
- board text added: "LM2662M - Negative Voltage Generator Inverting Charge Pump Converter Input: +VCC (1.5V-5.5V) Output: VEE (-VCC)"
- board text removed: "LM2662M - Negative Voltage Generator Inverting Charge Pump Converter Input: +VCC (1.5V-5.5V) Output: -VCC (~-VCC_IN)"
Changed lines of the file:
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@@
 	(net 3 "Net-(U1-CAP+)")
 	(net 4 "Net-(U1-CAP-)")
-	(net 5 "/LM2662M/VCCN")
+	(net 5 "/LM2662M/VEE")
 	(net 6 "Net-(J1-Pin_2)")
 	(net 7 "unconnected-(U1-FC-Pad1)")
@@
 			(layers "F.Cu" "F.Mask" "F.Paste")
 			(roundrect_rratio 0.25)
-			(net 5 "/LM2662M/VCCN")
+			(net 5 "/LM2662M/VEE")
 			(pintype "passive")
 		)
@@
 			(layers "*.Cu" "*.Mask")
 			(remove_unused_layers no)
-			(net 5 "/LM2662M/VCCN")
+			(net 5 "/LM2662M/VEE")
 			(pinfunction "Pin_1")
 			(pintype "passive")
@@
 			(layers "F.Cu" "F.Mask" "F.Paste")
 			(roundrect_rratio 0.25)
-			(net 5 "/LM2662M/VCCN")
+			(net 5 "/LM2662M/VEE")
 			(pintype "passive")
 		)
@@
 		)
 	)
-	(gr_text "LM2662M - Negative Voltage Generator\nInverting Charge Pump Converter\nInput: +VCC (1.5V-5.5V)\nOutput: -VCC (~-VCC_IN)\n\n"
+	(gr_text "LM2662M - Negative Voltage Generator\nInverting Charge Pump Converter\nInput: +VCC (1.5V-5.5V)\nOutput: VEE (-VCC)\n\n"
 		(at 141.99 85.19 0)
 		(layer "Dwgs.User")
