File: lm324drg4/lm324drg4.kicad_pcb (KiCad board)
At the start: 4 copper layers, 11 parts, among them U1 LM324DRG4

Commit message: [Rushil] changed vccn to vee
Connections:
- net /LM324DRG4/VCCN renamed /LM324DRG4/VEE
Changed lines of the file:
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@@
 	(net 1 "/LM324DRG4/VCC")
 	(net 2 "/LM324DRG4/GND")
-	(net 3 "/LM324DRG4/VCCN")
+	(net 3 "/LM324DRG4/VEE")
 	(net 4 "/LM324DRG4/PD0")
 	(net 5 "/LM324DRG4/OUT1")
@@
 			(layers "F.Cu" "F.Mask" "F.Paste")
 			(roundrect_rratio 0.25)
-			(net 3 "/LM324DRG4/VCCN")
+			(net 3 "/LM324DRG4/VEE")
 			(pintype "passive")
 		)
@@
 			(layers "F.Cu" "F.Mask" "F.Paste")
 			(roundrect_rratio 0.25)
-			(net 3 "/LM324DRG4/VCCN")
+			(net 3 "/LM324DRG4/VEE")
 			(pinfunction "GND")
 			(pintype "power_in")
