File: esp32-s3/block_esp32-s3.kicad_sch (KiCad schematic)
At the start: 27 parts, among them J1 DX07S016JA1R1500, SW1 RESET, SW2 BOOT, U1 ESP32-S3FN8, Y1 40Mhz

Commit message: [Rushil] added ldo
Parts:
- added C18, C19: 22uF, Capacitor_SMD:C_0603_1608Metric, symbol Library:C
- added D1: LED, LED_SMD:LED_0603_1608Metric_Pad1.05x0.95mm_HandSolder, symbol Library:LED
- added R3: 4.7K, Resistor_SMD:R_0603_1608Metric, symbol Library:R
- added U2: AP2112K-3.3, Package_TO_SOT_SMD:SOT-23-5, symbol Regulator_Linear:AP2112K-3.3
Connections:
- net 3V3: now also C19.1, R3.1, U2.5 (VOUT)
- net GND: now also C18.2, C19.2, D1.1 (K), U2.2 (GND)
- net VBUS: now reaches J1.11 (VBUS), J1.2 (VBUS)
- net VBUS: now also C18.1, U2.1 (VIN), U2.3 (EN)
- new net: D1.2 (A), R3.2
- no-connect marks 5 -> 4
Other:
- note added: "3.3 V Low Dropout Linear Regulator Input: 2.5 V - 6 V Output: Fixed 3.3 V, up to 600 mA"

Commit message: [Rushil] some minor changes
Parts:
- added R4, R5: 5.1K, Resistor_SMD:R_0603_1608Metric_Pad0.98x0.95mm_HandSolder, symbol Device:R
Connections:
- net GND: now also R4.2, R5.1
- net at J1.3 (CC1): now also R5.2
- net at J1.9 (CC2): now also R4.1
- no-connect marks 4 -> 2
Changed lines of the file:
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@@
 		(at 20.32 96.52)
 	)
-	(no_connect
-		(at 20.32 99.06)
-	)
-	(no_connect
-		(at 20.32 86.36)
-	)
 	(wire
 		(pts
@@
 	(wire
 		(pts
+			(xy 17.78 99.06) (xy 17.78 100.33)
+		)
+		(stroke
+			(width 0)
+			(type default)
+		)
+	)
+	(wire
+		(pts
 			(xy 64.77 110.49) (xy 67.31 110.49)
 		)
@@
 	(wire
 		(pts
+			(xy 17.78 86.36) (xy 20.32 86.36)
+		)
+		(stroke
+			(width 0)
+			(type default)
+		)
+	)
+	(wire
+		(pts
 			(xy 77.47 110.49) (xy 77.47 111.76)
 		)
@@
 	(wire
 		(pts
+			(xy 20.32 99.06) (xy 17.78 99.06)
+		)
+		(stroke
+			(width 0)
+			(type default)
+		)
+	)
+	(wire
+		(pts
 			(xy 160.02 53.34) (xy 160.02 52.07)
 		)
@@
 		)
 	)
+	(hierarchical_label "GND"
+		(shape input)
+		(at 17.78 107.95 270)
+		(effects
+			(font
+				(size 1.27 1.27)
+			)
+			(justify right)
+		)
+	)
 	(hierarchical_label "SPIHD"
 		(shape input)
@@
 		)
 	)
+	(hierarchical_label "GND"
+		(shape input)
+		(at 17.78 78.74 90)
+		(effects
+			(font
+				(size 1.27 1.27)
+			)
+			(justify left)
+		)
+	)
 	(hierarchical_label "GPIO14"
 		(shape input)
@@
 	)
 	(symbol
+		(lib_id "Device:R")
+		(at 17.78 104.14 0)
+		(unit 1)
+		(exclude_from_sim no)
+		(in_bom yes)
+		(on_board yes)
+		(dnp no)
+		(property "Reference" "R4"
+			(at 19.05 104.14 0)
+			(effects
+				(font
+					(size 1.27 1.27)
+				)
+				(justify left)
+			)
+		)
+		(property "Value" "5.1K"
+			(at 18.034 106.172 90)
+			(effects
+				(font
+					(size 1.27 1.27)
+				)
+				(justify left)
+			)
+		)
+		(property "Footprint" "Resistor_SMD:R_0603_1608Metric_Pad0.98x0.95mm_HandSolder"
+			(at 16.002 104.14 90)
+			(effects
+				(font
+					(size 1.27 1.27)
+				)
+				(hide yes)
+			)
+		)
+		(property "Datasheet" "~"
+			(at 17.78 104.14 0)
+			(effects
+				(font
+					(size 1.27 1.27)
+				)
+				(hide yes)
+			)
+		)
+		(property "Description" ""
+			(at 17.78 104.14 0)
+			(effects
+				(font
+					(size 1.27 1.27)
+				)
+			)
+		)
+		(property "LCSC" "C14677"
+			(at 17.78 104.14 0)
+			(effects
+				(font
+					(size 1.27 1.27)
+				)
+				(hide yes)
+			)
+		)
+		(property "MPN" "RC0603JR-075K1L"
+			(at 17.78 104.14 0)
+			(effects
+				(font
+					(size 1.27 1.27)
+				)
+				(hide yes)
+			)
+		)
+		(pin "1"
+		)
+		(pin "2"
+		)
+		(instances
+			(project "esp32-s3"
+				(path "/ee0fcbb6-6e07-467d-8954-b6df91be3afa/38c500d9-8c49-47a3-ac44-6b9512864f40"
+					(reference "R4")
+					(unit 1)
+				)
+			)
+		)
+	)
+	(symbol
 		(lib_id "Regulator_Linear:AP2112K-3.3")
 		(at 255.27 49.53 0)
@@
 					(unit 1)
 				)
+			)
+		)
+	)
+	(symbol
+		(lib_id "Device:R")
+		(at 17.78 82.55 0)
+		(unit 1)
+		(exclude_from_sim no)
+		(in_bom yes)
+		(on_board yes)
+		(dnp no)
+		(property "Reference" "R5"
+			(at 19.05 82.55 0)
+			(effects
+				(font
+					(size 1.27 1.27)
+				)
+				(justify left)
+			)
+		)
+		(property "Value" "5.1K"
+			(at 17.78 85.09 90)
+			(effects
+				(font
+					(size 1.27 1.27)
+				)
+				(justify left)
+			)
+		)
+		(property "Footprint" "Resistor_SMD:R_0603_1608Metric_Pad0.98x0.95mm_HandSolder"
+			(at 16.002 82.55 90)
+			(effects
+				(font
+					(size 1.27 1.27)
+				)
+				(hide yes)
+			)
+		)
+		(property "Datasheet" "~"
+			(at 17.78 82.55 0)
+			(effects
+				(font
+					(size 1.27 1.27)
+				)
+				(hide yes)
+			)
+		)
+		(property "Description" ""
+			(at 17.78 82.55 0)
+			(effects
+				(font
+					(size 1.27 1.27)
+				)
+			)
+		)
+		(property "LCSC" "C14677"
+			(at 17.78 82.55 0)
+			(effects
+				(font
+					(size 1.27 1.27)
+				)
+				(hide yes)
+			)
+		)
+		(property "MPN" "RC0603JR-075K1L"
+			(at 17.78 82.55 0)
+			(effects
+				(font
+					(size 1.27 1.27)
+				)
+				(hide yes)
+			)
+		)
+		(pin "1"
+		)
+		(pin "2"
+		)
+		(instances
+			(project "esp32-s3"
+				(path "/ee0fcbb6-6e07-467d-8954-b6df91be3afa/38c500d9-8c49-47a3-ac44-6b9512864f40"
+					(reference "R5")
+					(unit 1)
+				)
