File: esp32-s3/esp32-s3.kicad_pcb (KiCad board)
At the start: 4 copper layers, 27 parts, among them J1 DX07S016JA1R1500, SW1 RESET, SW2 BOOT, U1 ESP32-S3FN8, Y1 40Mhz

Commit message: [Rushil] added ldo
Parts:
- added C18: 22uF, Capacitor_SMD:C_0603_1608Metric, F.Cu at (150.1, 109.9)
- added C19: 22uF, Capacitor_SMD:C_0603_1608Metric, F.Cu at (153.3, 107.3)
- added D1: LED, LED_SMD:LED_0603_1608Metric_Pad1.05x0.95mm_HandSolder, F.Cu at (156.6, 107.3)
- added R3: 4.7K, Resistor_SMD:R_0603_1608Metric, F.Cu at (156.7, 109.0)
- added U2: AP2112K-3.3, Package_TO_SOT_SMD:SOT-23-5, F.Cu at (153.0, 110.0)
- moved C5 2.07 mm to (158.3, 121.4)
- moved C6 2.07 mm to (159.9, 121.4)
- moved C17 0.69 mm to (156.8, 111.0)
- moved R2 0.69 mm to (156.8, 112.5)
- moved C9 0.17 mm to (156.6, 115.1)
Connections:
- J1 pad 11: unconnected-(J1-VBUS-Pad11) -> /ESP32-S3/VBUS
- J1 pad 2: unconnected-(J1-VBUS-Pad11)_1 -> /ESP32-S3/VBUS
Routing:
- net /ESP32-S3/3V3: track 6.49 -> 24.5 mm, vias 2 -> 3
- net /ESP32-S3/GND: track 7.59 -> 20.6 mm
- net Net-(D1-A): track 0.00 -> 1.71 mm
- net /ESP32-S3/VDD_SPI: track 4.64 -> 3.30 mm
- net /ESP32-S3/VBUS: vias 0 -> 16
- added copper zone on F.Cu, net /ESP32-S3/VBUS
- added copper zone on In2.Cu, net /ESP32-S3/VBUS
Other:
- board text added: "LDO"

Commit message: [Rushil] some minor changes
Parts:
- added R4: 5.1K, Resistor_SMD:R_0603_1608Metric_Pad0.98x0.95mm_HandSolder, F.Cu at (153.5, 118.8)
- added R5: 5.1K, Resistor_SMD:R_0603_1608Metric_Pad0.98x0.95mm_HandSolder, F.Cu at (153.2, 114.5)
Connections:
- J1 pad 3: unconnected-(J1-CC1-Pad3) -> Net-(J1-CC1)
- J1 pad 9: unconnected-(J1-CC2-Pad9) -> Net-(J1-CC2)
Routing:
- net Net-(J1-CC1): track 0.00 -> 2.76 mm
- net Net-(J1-CC2): track 0.00 -> 1.59 mm
- net /ESP32-S3/GND: vias 41 -> 39
